File: nightLight.brd (EAGLE design)
At the start: 46.6 x 55.9 mm, 14 parts

Commit message: Working on hooking up MQ-07 CO sensor
Parts:
- added C2, C3: 10uF, SparkFun-Capacitors:CPOL-RADIAL-2.5MM-5MM
- added Q1: 200mA/40V, SparkFun-DiscreteSemi:TO-92-EZ
- added R5: 10k, SparkFun-Resistors:AXIAL-0.3
Connections:
- new net A1: GS1.B1, JP1.11, JP1.A1, R5.P$1
- net 5V: now also GS1.A1
- net GND: now also R5.P$2
Routing:
- net D6: track 12.9 -> 0.91 mm
- net D2: track 9.87 -> 4.02 mm
Changed lines of the file:
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@@
 <attribute name="VALUE" x="16.27" y="12.455" size="1.27" layer="27"/>
+</element>
+<element name="Q1" library="SparkFun-DiscreteSemi" package="TO-92-EZ" value="200mA/40V" x="44.45" y="50.8">
+<attribute name="NAME" x="44.45" y="53.848" size="0.6096" layer="25" font="vector" ratio="20" align="bottom-center"/>
+<attribute name="PROD_ID" value="TRANS-08447" x="44.45" y="50.8" size="1.778" layer="27" display="off"/>
+<attribute name="VALUE" x="44.45" y="48.895" size="0.6096" layer="27" font="vector" ratio="20" align="top-center"/>
+</element>
+<element name="C2" library="SparkFun-Capacitors" package="CPOL-RADIAL-2.5MM-5MM" value="10uF" x="-110.49" y="24.13">
+<attribute name="NAME" x="-110.49" y="26.797" size="0.6096" layer="25" font="vector" ratio="20" align="bottom-center"/>
+<attribute name="PROD_ID" value="CAP-08440" x="-110.49" y="24.13" size="1.778" layer="27" display="off"/>
+<attribute name="VALUE" x="-110.49" y="21.463" size="0.6096" layer="27" font="vector" ratio="20" align="top-center"/>
+</element>
+<element name="C3" library="SparkFun-Capacitors" package="CPOL-RADIAL-2.5MM-5MM" value="10uF" x="-116.84" y="24.13">
+<attribute name="NAME" x="-116.84" y="26.797" size="0.6096" layer="25" font="vector" ratio="20" align="bottom-center"/>
+<attribute name="PROD_ID" value="CAP-08440" x="-116.84" y="24.13" size="1.778" layer="27" display="off"/>
+<attribute name="VALUE" x="-116.84" y="21.463" size="0.6096" layer="27" font="vector" ratio="20" align="top-center"/>
+</element>
+<element name="R5" library="SparkFun-Resistors" package="AXIAL-0.3" value="10k" x="39.37" y="45.72" rot="R90">
+<attribute name="NAME" x="38.354" y="45.72" size="0.6096" layer="25" font="vector" ratio="20" rot="R90" align="bottom-center"/>
+<attribute name="PROD_ID" value="RES-08375" x="39.37" y="45.72" size="1.778" layer="27" rot="R90" display="off"/>
+<attribute name="VALUE" x="40.386" y="45.72" size="0.6096" layer="27" font="vector" ratio="20" rot="R90" align="top-center"/>
 </element>
 </elements>
@@
 <contactref element="C1" pad="-"/>
 <wire x1="26.67" y1="69.9516" x2="26.67" y2="69.85" width="0.1524" layer="16"/>
+<contactref element="R5" pad="P$2"/>
 <wire x1="26.67" y1="69.9516" x2="33.06" y2="74.93" width="0" layer="19" extent="1-1"/>
 <wire x1="24.13" y1="69.85" x2="26.67" y2="69.9516" width="0" layer="19" extent="1-1"/>
@@
 <wire x1="17.54" y1="35.95" x2="36.83" y2="49.53" width="0" layer="19" extent="1-1"/>
 <wire x1="19.1931375" y1="31.769340625" x2="17.54" y2="35.95" width="0" layer="19" extent="1-1"/>
+<wire x1="39.37" y1="49.53" x2="3.81" y2="74.93" width="0" layer="19" extent="1-1"/>
 </signal>
 <signal name="5V">
@@
 <contactref element="VDD" pad="1"/>
 <contactref element="C1" pad="+"/>
-<wire x1="6.4008" y1="77.5716" x2="38.06" y2="74.93" width="0" layer="19" extent="1-1"/>
+<contactref element="GS1" pad="A1"/>
+<wire x1="34.75" y1="64.31" x2="38.06" y2="74.93" width="0" layer="19" extent="1-1"/>
+<wire x1="6.35" y1="77.47" x2="34.75" y2="64.31" width="0" layer="19" extent="1-1"/>
 <wire x1="3.81" y1="77.47" x2="6.35" y2="77.47" width="0" layer="19" extent="1-1"/>
-<wire x1="17.283065625" y1="27.6088" x2="6.35" y2="77.47" width="0" layer="19" extent="1-1"/>
+<wire x1="17.283065625" y1="27.6088" x2="34.75" y2="64.31" width="0" layer="19" extent="1-1"/>
 </signal>
 <signal name="A0">
@@
 <contactref element="JP1" pad="D2"/>
 <wire x1="26.67" y1="54.5592" x2="26.67" y2="54.61" width="0.1524" layer="16"/>
-<wire x1="25.4508" y1="48.9204" x2="25.6032" y2="48.768" width="0.1524" layer="1"/>
-<wire x1="25.4508" y1="54.5592" x2="25.4508" y2="48.9204" width="0.1524" layer="1"/>
 <wire x1="25.4508" y1="54.5592" x2="24.13" y2="54.61" width="0.1524" layer="1"/>
 <wire x1="26.67" y1="54.7116" x2="26.67" y2="54.61" width="0.1524" layer="1"/>
 <wire x1="26.67" y1="54.7116" x2="24.13" y2="54.61" width="0.1524" layer="1"/>
-<wire x1="25.6032" y1="48.768" x2="34.29" y2="49.53" width="0" layer="19" extent="1-1"/>
+<wire x1="26.67" y1="54.5592" x2="34.29" y2="49.53" width="0" layer="19" extent="16-16"/>
 <wire x1="38.1" y1="31.75" x2="34.29" y2="49.53" width="0" layer="19" extent="1-1"/>
 </signal>
@@
 <contactref element="JP1" pad="D6"/>
 <wire x1="30.9372" y1="49.53" x2="31.75" y2="49.53" width="0.1524" layer="16"/>
-<wire x1="25.4508" y1="63.5508" x2="25.4508" y2="54.102" width="0.1524" layer="16"/>
 <wire x1="24.2316" y1="64.77" x2="24.13" y2="64.77" width="0.1524" layer="16"/>
-<wire x1="26.67" y1="64.77" x2="24.13" y2="64.77" width="0.1524" layer="1"/>
-<wire x1="25.4508" y1="63.5508" x2="26.67" y2="64.77" width="0" layer="19" extent="16-16"/>
-<wire x1="30.9372" y1="49.53" x2="25.4508" y2="54.102" width="0" layer="19" extent="16-16"/>
+<wire x1="24.2316" y1="64.77" x2="26.67" y2="64.77" width="0" layer="19" extent="16-16"/>
+<wire x1="30.9372" y1="49.53" x2="26.67" y2="64.77" width="0" layer="19" extent="16-16"/>
+</signal>
+<signal name="A1">
+<contactref element="GS1" pad="B1"/>
+<contactref element="R5" pad="P$1"/>
+<contactref element="JP1" pad="A1"/>
+<contactref element="JP1" pad="11"/>
+<wire x1="6.35" y1="52.07" x2="41.45" y2="64.31" width="0" layer="19" extent="1-1"/>
+<wire x1="3.81" y1="52.07" x2="6.35" y2="52.07" width="0" layer="19" extent="1-1"/>
+<wire x1="39.37" y1="41.91" x2="3.81" y2="52.07" width="0" layer="19" extent="1-1"/>
 </signal>
 </signals>
