File: nightLight.sch (EAGLE design)
At the start: 14 parts

Commit message: Working on hooking up MQ-07 CO sensor
Parts:
- added C2, C3: 10uF, SparkFun-Capacitors:10UF-POLAR-RADIAL-2.5MM-25V-20%
- added Q1: 200mA/40V, SparkFun-DiscreteSemi:TRANS_NPN-2N3904-EZ
- added R5: 10k, SparkFun-Resistors:10KOHM-HORIZ-1/6W-5%
Connections:
- new net A1: GS1.B1, JP1.A1, R5.1
- net 5V: now also GS1.A1
- net GND: now also R5.2
Changed lines of the file:
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@@
 <part name="GND" library="NeoPixelRing" deviceset="PINHD-1X1" device="CB"/>
 <part name="GND_2" library="NeoPixelRing" deviceset="PINHD-1X1" device="CB"/>
+<part name="Q1" library="SparkFun-DiscreteSemi" deviceset="TRANS_NPN" device="-2N3904-EZ" value="200mA/40V"/>
+<part name="C2" library="SparkFun-Capacitors" deviceset="10UF-POLAR" device="-RADIAL-2.5MM-25V-20%" value="10uF"/>
+<part name="C3" library="SparkFun-Capacitors" deviceset="10UF-POLAR" device="-RADIAL-2.5MM-25V-20%" value="10uF"/>
+<part name="R5" library="SparkFun-Resistors" deviceset="10KOHM" device="-HORIZ-1/6W-5%" value="10k"/>
 </parts>
 <sheets>
@@
 <attribute name="NAME" x="3.81" y="37.465" size="1.778" layer="95" rot="R180"/>
 <attribute name="VALUE" x="3.81" y="45.72" size="1.778" layer="96" rot="R180"/>
+</instance>
+<instance part="Q1" gate="G$1" x="71.12" y="129.54">
+<attribute name="NAME" x="73.66" y="129.54" size="1.778" layer="95" font="vector"/>
+<attribute name="VALUE" x="73.66" y="127.254" size="1.778" layer="96" font="vector"/>
+</instance>
+<instance part="C2" gate="G$1" x="104.14" y="137.16">
+<attribute name="NAME" x="105.156" y="137.795" size="1.778" layer="95" font="vector"/>
+<attribute name="VALUE" x="105.156" y="132.969" size="1.778" layer="96" font="vector"/>
+</instance>
+<instance part="C3" gate="G$1" x="53.34" y="137.16">
+<attribute name="NAME" x="54.356" y="137.795" size="1.778" layer="95" font="vector"/>
+<attribute name="VALUE" x="54.356" y="132.969" size="1.778" layer="96" font="vector"/>
+</instance>
+<instance part="R5" gate="G$1" x="99.06" y="149.86">
+<attribute name="NAME" x="99.06" y="151.384" size="1.778" layer="95" font="vector" align="bottom-center"/>
+<attribute name="VALUE" x="99.06" y="148.336" size="1.778" layer="96" font="vector" align="top-center"/>
 </instance>
 </instances>
@@
 <junction x="10.16" y="43.18"/>
 <label x="40.64" y="43.18" size="1.778" layer="95"/>
+</segment>
+<segment>
+<pinref part="R5" gate="G$1" pin="2"/>
+<wire x1="104.14" y1="149.86" x2="109.22" y2="149.86" width="0.1524" layer="91"/>
+<label x="111.76" y="149.86" size="1.778" layer="95"/>
 </segment>
 </net>
@@
 <label x="40.64" y="60.96" size="1.778" layer="95"/>
 </segment>
+<segment>
+<pinref part="GS1" gate="G$1" pin="A1"/>
+<wire x1="68.58" y1="149.86" x2="63.5" y2="149.86" width="0.1524" layer="91"/>
+<label x="58.42" y="149.86" size="1.778" layer="95"/>
+</segment>
 </net>
 <net name="A0" class="0">
@@
 </segment>
 </net>
+<net name="A1" class="0">
+<segment>
+<pinref part="GS1" gate="G$1" pin="B1"/>
+<pinref part="R5" gate="G$1" pin="1"/>
+<wire x1="88.9" y1="149.86" x2="91.44" y2="149.86" width="0.1524" layer="91"/>
+<wire x1="91.44" y1="149.86" x2="93.98" y2="149.86" width="0.1524" layer="91"/>
+<wire x1="91.44" y1="149.86" x2="91.44" y2="154.94" width="0.1524" layer="91"/>
+<wire x1="91.44" y1="154.94" x2="93.98" y2="154.94" width="0.1524" layer="91"/>
+<junction x="91.44" y="149.86"/>
+<label x="99.06" y="154.94" size="1.778" layer="95"/>
+</segment>
+<segment>
+<pinref part="JP1" gate="G$1" pin="A1"/>
+<wire x1="119.38" y1="55.88" x2="114.3" y2="55.88" width="0.1524" layer="91"/>
+<label x="109.22" y="55.88" size="1.778" layer="95"/>
+</segment>
+</net>

Commit message: Finished MQ07 Hookup
Connections:
- new net D3: JP1.(JTAG_TRST)D3, Q1.B
- new net N$2: C3.-, GS1.H2, Q1.C
- net 3V3: now also C2.+, GS1.A1
- net 5V: now also C3.+, GS1.H1; no longer GS1.A1
- net A1: now also C2.-
- net GND: now also Q1.E
Other:
- moved on the sheet: C2, C3
Changed lines of the file:
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@@
 <attribute name="VALUE" x="73.66" y="127.254" size="1.778" layer="96" font="vector"/>
 </instance>
-<instance part="C2" gate="G$1" x="104.14" y="137.16">
-<attribute name="NAME" x="105.156" y="137.795" size="1.778" layer="95" font="vector"/>
-<attribute name="VALUE" x="105.156" y="132.969" size="1.778" layer="96" font="vector"/>
-</instance>
-<instance part="C3" gate="G$1" x="53.34" y="137.16">
-<attribute name="NAME" x="54.356" y="137.795" size="1.778" layer="95" font="vector"/>
-<attribute name="VALUE" x="54.356" y="132.969" size="1.778" layer="96" font="vector"/>
+<instance part="C2" gate="G$1" x="78.74" y="157.48" rot="R90">
+<attribute name="NAME" x="78.105" y="158.496" size="1.778" layer="95" font="vector" rot="R90"/>
+<attribute name="VALUE" x="82.931" y="158.496" size="1.778" layer="96" font="vector" rot="R90"/>
+</instance>
+<instance part="C3" gate="G$1" x="63.5" y="142.24">
+<attribute name="NAME" x="64.516" y="142.875" size="1.778" layer="95" font="vector"/>
+<attribute name="VALUE" x="64.516" y="138.049" size="1.778" layer="96" font="vector"/>
 </instance>
 <instance part="R5" gate="G$1" x="99.06" y="149.86">
@@
 <wire x1="104.14" y1="149.86" x2="109.22" y2="149.86" width="0.1524" layer="91"/>
 <label x="111.76" y="149.86" size="1.778" layer="95"/>
+</segment>
+<segment>
+<pinref part="Q1" gate="G$1" pin="E"/>
+<wire x1="73.66" y1="124.46" x2="73.66" y2="121.92" width="0.1524" layer="91"/>
+<wire x1="73.66" y1="121.92" x2="83.82" y2="121.92" width="0.1524" layer="91"/>
+<label x="86.36" y="121.92" size="1.778" layer="95"/>
 </segment>
 </net>
@@
 </segment>
 <segment>
-<pinref part="GS1" gate="G$1" pin="A1"/>
-<wire x1="68.58" y1="149.86" x2="63.5" y2="149.86" width="0.1524" layer="91"/>
-<label x="58.42" y="149.86" size="1.778" layer="95"/>
+<pinref part="GS1" gate="G$1" pin="H1"/>
+<wire x1="68.58" y1="147.32" x2="63.5" y2="147.32" width="0.1524" layer="91"/>
+<label x="58.42" y="147.32" size="1.778" layer="95"/>
+<pinref part="C3" gate="G$1" pin="+"/>
+<wire x1="63.5" y1="144.78" x2="63.5" y2="147.32" width="0.1524" layer="91"/>
 </segment>
 </net>
@@
 <junction x="7.62" y="91.44"/>
 <label x="15.24" y="91.44" size="1.778" layer="95"/>
+</segment>
+<segment>
+<pinref part="GS1" gate="G$1" pin="A1"/>
+<wire x1="68.58" y1="149.86" x2="63.5" y2="149.86" width="0.1524" layer="91"/>
+<label x="58.42" y="149.86" size="1.778" layer="95"/>
+<wire x1="68.58" y1="149.86" x2="68.58" y2="157.48" width="0.1524" layer="91"/>
+<junction x="68.58" y="149.86"/>
+<pinref part="C2" gate="G$1" pin="+"/>
+<wire x1="68.58" y1="157.48" x2="76.2" y2="157.48" width="0.1524" layer="91"/>
 </segment>
 </net>
@@
 <junction x="91.44" y="149.86"/>
 <label x="99.06" y="154.94" size="1.778" layer="95"/>
+<pinref part="C2" gate="G$1" pin="-"/>
+<wire x1="83.82" y1="157.48" x2="88.9" y2="157.48" width="0.1524" layer="91"/>
+<wire x1="88.9" y1="157.48" x2="88.9" y2="149.86" width="0.1524" layer="91"/>
+<junction x="88.9" y="149.86"/>
 </segment>
 <segment>
@@
 </segment>
 </net>
+<net name="N$2" class="0">
+<segment>
+<pinref part="GS1" gate="G$1" pin="H2"/>
+<wire x1="88.9" y1="147.32" x2="88.9" y2="134.62" width="0.1524" layer="91"/>
+<pinref part="Q1" gate="G$1" pin="C"/>
+<wire x1="88.9" y1="134.62" x2="73.66" y2="134.62" width="0.1524" layer="91"/>
+<pinref part="C3" gate="G$1" pin="-"/>
+<wire x1="63.5" y1="137.16" x2="63.5" y2="134.62" width="0.1524" layer="91"/>
+<wire x1="63.5" y1="134.62" x2="73.66" y2="134.62" width="0.1524" layer="91"/>
+<junction x="73.66" y="134.62"/>
+</segment>
+</net>
+<net name="D3" class="0">
+<segment>
+<pinref part="Q1" gate="G$1" pin="B"/>
+<wire x1="68.58" y1="129.54" x2="63.5" y2="129.54" width="0.1524" layer="91"/>
+<label x="60.96" y="129.54" size="1.778" layer="95"/>
+</segment>
+<segment>
+<pinref part="JP1" gate="G$1" pin="(JTAG_TRST)D3"/>
+<wire x1="162.56" y1="60.96" x2="170.18" y2="60.96" width="0.1524" layer="91"/>
+<label x="172.72" y="60.96" size="1.778" layer="95"/>
+</segment>
+</net>

Commit message: This is the board i ordered
Parts:
- removed FRAME1: FRAME-LETTER, SparkFun-Aesthetics:FRAME-LETTER
Connections:
- new net A5: JP1.A5(SPI1_MOSI), R2.1, R3.P$2
- net A0: no longer R2.1, R3.P$2
Changed lines of the file:
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@@
 <part name="J1" library="SparkFun-Connectors" deviceset="CONN_04" device=""/>
 <part name="R4" library="SparkFun-Resistors" deviceset="10KOHM" device="-HORIZ-1/4W-1%" value="10k"/>
-<part name="FRAME1" library="SparkFun-Aesthetics" deviceset="FRAME-LETTER" device=""/>
 <part name="GS1" library="SparkFun-Sensors" deviceset="GAS_SENSOR" device="MQ-3"/>
 <part name="DIN" library="NeoPixelRing" deviceset="PINHD-1X1" device="CB"/>
@@
 <attribute name="VALUE" x="9.144" y="96.52" size="1.778" layer="96" font="vector" rot="R90" align="top-center"/>
 </instance>
-<instance part="FRAME1" gate="G$1" x="-15.24" y="-20.32"/>
-<instance part="FRAME1" gate="V" x="132.08" y="-20.32">
-<attribute name="LAST_DATE_TIME" x="144.78" y="-19.05" size="2.54" layer="94" font="vector"/>
-<attribute name="SHEET" x="218.44" y="-19.05" size="2.54" layer="94" font="vector"/>
-<attribute name="DRAWING_NAME" x="147.574" y="-2.54" size="2.7432" layer="94" font="vector"/>
-<attribute name="DESIGNER" x="155.194" y="-9.144" size="2.7432" layer="94" font="vector"/>
-<attribute name="REV" x="220.98" y="-13.716" size="2.7432" layer="94" font="vector"/>
-</instance>
 <instance part="GS1" gate="G$1" x="78.74" y="147.32">
 <attribute name="NAME" x="71.12" y="152.654" size="1.778" layer="95" font="vector"/>
@@
 <wire x1="119.38" y1="53.34" x2="114.3" y2="53.34" width="0.1524" layer="91"/>
 <label x="109.22" y="53.34" size="1.778" layer="95"/>
-</segment>
-<segment>
-<pinref part="R3" gate="G$1" pin="P$2"/>
-<pinref part="R2" gate="G$1" pin="1"/>
-<wire x1="-5.08" y1="142.24" x2="-5.08" y2="134.62" width="0.1524" layer="91"/>
-<wire x1="-5.08" y1="142.24" x2="-5.08" y2="137.16" width="0.1524" layer="91"/>
-<junction x="-5.08" y="142.24"/>
-<wire x1="-5.08" y1="137.16" x2="7.62" y2="137.16" width="0.1524" layer="91"/>
-<label x="10.16" y="137.16" size="1.778" layer="95"/>
 </segment>
 </net>
@@
 </segment>
 </net>
+<net name="A5" class="0">
+<segment>
+<pinref part="R3" gate="G$1" pin="P$2"/>
+<pinref part="R2" gate="G$1" pin="1"/>
+<wire x1="-5.08" y1="142.24" x2="-5.08" y2="134.62" width="0.1524" layer="91"/>
+<wire x1="-5.08" y1="142.24" x2="-5.08" y2="137.16" width="0.1524" layer="91"/>
+<junction x="-5.08" y="142.24"/>
+<wire x1="-5.08" y1="137.16" x2="7.62" y2="137.16" width="0.1524" layer="91"/>
+<label x="10.16" y="137.16" size="1.778" layer="95"/>
+</segment>
+<segment>
+<pinref part="JP1" gate="G$1" pin="A5(SPI1_MOSI)"/>
+<wire x1="119.38" y1="66.04" x2="114.3" y2="66.04" width="0.1524" layer="91"/>
+<label x="109.22" y="66.04" size="1.778" layer="95"/>
+</segment>
+</net>
